File: Hardware/Electronics/Schematic/woodenClock.sch (KiCad schematic (older format))
At the start: 41 parts, among them P1 CONN_02X08, U1 TLC59208F, U2 TLC59208F, U3 TLC59208F, U4 TLC59208F

Commit message: Changed dispaly board schematic and layout version to 1.0.0 Moved vias from the capacitor pads Added github link on the silkscreen Changed files architecture Pushed new gerbers
Parts:
- removed C1, C2, C3, C4: 100n, Capacitors_SMD:C_0402_NoSilk, symbol device:C_Small
- removed P1: CONN_02X08, kicad-libraries-master:Pin_Header_Straight_2x08_Pitch2.54mm_SMD, symbol conn:CONN_02X08
- removed R1, R10, R11, R12, R13, R14, R15, R16, R17, R18, R19, R2, R20, R21, R22, R23, R24, R25, R26, R27, R28, R29, R3, R30, R31, R32, R4, R5, R6, R7, R8, R9: 47, Resistors_SMD:R_0805_HandSoldering, symbol device:R
- removed U1, U2, U3, U4: TLC59208F, kicad-libraries-master:TSSOP16, symbol texas:TLC59208F
Connections:
- net labels removed: +3.3V, C1, C10, C11, C12, C13, C14, C15, C16, C17, C18, C19, C2, C20, C21, C22, C23, C24, C25, C26, C27, C28, C29, C3, C30, C31, C32, C4, C5, C6, C7, C8, C9, CLK, GND, LAT, OE, R1, R10, R11, R12, R13, R14, R15, R16, R17, R18, R19, R2, R20, R21, R22, R23, R24, R25, R26, R27, R28, R29, R3, R30, R31, R32, R4, R5, R6, R7, R8, R9, RESET, RST, SCL1, SCL2, SCL3, SCL4, SDA1, SDA2, SDA3, SDA4, SIN
- wire segments 276 -> 0

Commit message: Schematic update -- start of the main board designe
Changed lines of the file:
@@
 EESchema Schematic File Version 4
-LIBS:main-cache
 EELAYER 26 0
 EELAYER END
 $Descr A4 11693 8268
 encoding utf-8
-Sheet 1 7
+Sheet 1 8
 Title "Wooden clock"
 Date "2018-10-21"
@@
 F0 "DisplayBoard" 50
 F1 "DisplayBoard/DisplayBoard.sch" 50
-F2 "SDA1" I L 8150 3000 50
-F3 "SCL1" B L 8150 3100 50
-F4 "SDA2" I L 8150 3250 50
-F5 "SDA3" I L 8150 3500 50
-F6 "SDA4" I L 8150 3750 50
+F2 "SDA1" B L 8150 3000 50
+F3 "SCL1" I L 8150 3100 50
+F4 "SDA2" B L 8150 3250 50
+F5 "SDA3" B L 8150 3500 50
+F6 "SDA4" B L 8150 3750 50
 F7 "OUTPUT_ENABLE" I L 8150 4500 50
 F8 "LATCH" I L 8150 4400 50
@@
 F13 "3V3" U L 8150 4800 50
 F14 "GND" U L 8150 4900 50
-F15 "SCL2" B L 8150 3350 50
-F16 "SCL3" B L 8150 3600 50
-F17 "SCL4" B L 8150 3850 50
+F15 "SCL2" I L 8150 3350 50
+F16 "SCL3" I L 8150 3600 50
+F17 "SCL4" I L 8150 3850 50
 $EndSheet
+$Sheet
+S 4950 2900 1800 2150
+U 5CCD8EC9
+F0 "MainBoard" 50
+F1 "MainBoard/MainBoard.sch" 50
+F2 "SDA1" B R 6750 3000 50
+F3 "SCL1" O R 6750 3100 50
+F4 "SDA2" B R 6750 3250 50
+F5 "SCL2" O R 6750 3350 50
+F6 "SDA3" B R 6750 3500 50
+F7 "SCL3" O R 6750 3600 50
+F8 "SDA4" B R 6750 3750 50
+F9 "SCL4" O R 6750 3850 50
+F10 "I2C_RESET" O R 6750 4000 50
+F11 "DATA_IN" O R 6750 4200 50
+F12 "CLK" O R 6750 4300 50
+F13 "LATCH" O R 6750 4400 50
+F14 "OUTPUT_ENABLE" O R 6750 4500 50
+F15 "ROW_RESET" O R 6750 4600 50
+F16 "3V3" U R 6750 4800 50
+F17 "GND" U R 6750 4900 50
+$EndSheet
+Wire Wire Line
+	6750 3000 8150 3000
+Wire Wire Line
+	8150 3100 6750 3100
+Wire Wire Line
+	6750 3250 8150 3250
+Wire Wire Line
+	8150 3350 6750 3350
+Wire Wire Line
+	6750 3500 8150 3500
+Wire Wire Line
+	8150 3600 6750 3600
+Wire Wire Line
+	6750 3750 8150 3750
+Wire Wire Line
+	8150 3850 6750 3850
+Wire Wire Line
+	6750 4000 8150 4000
+Wire Wire Line
+	6750 4200 8150 4200
+Wire Wire Line
+	6750 4300 8150 4300
+Wire Wire Line
+	6750 4400 8150 4400
+Wire Wire Line
+	6750 4500 8150 4500
+Wire Wire Line
+	6750 4600 8150 4600
+Wire Wire Line
+	6750 4800 8150 4800
+Wire Wire Line
+	6750 4900 8150 4900
 $EndSCHEMATC
