File: Hardware/Electronics/Layout/ButtonBoard/ButtonBoard.kicad_pcb (KiCad board)
At the start: 2 copper layers, 67 x 88 mm, 10 parts, among them P11 CONN_01X03, U16 TTP223

Commit message: updated schematics
Other:
- net class Default removed
