File: Hardware/Electronics/Schematic/ButtonBoard/ButtonBoard.kicad_sch (KiCad schematic)
At the start: 6 parts, among them P11 CONN_01X03, U16 TTP223

Commit message: Kicad files cleanup
Parts:
- gave numbers to parts that had none: 2
