File: Hardware/Electronics/Schematic/DisplayBoard/MosfetMultiplexer/MosfetMultiplexer.kicad_sch (KiCad schematic)
At the start: 26 parts

Commit message: Kicad files cleanup
Parts:
- removed ?: 74HC595, kicad-libraries-master:TSSOP16, symbol 74xx1:74HC595
- added U5: 74HC595, symbol 74xx:74HC595
- gave numbers to parts that had none: 25
Connections:
- net +3.3V: now also U5.16 (VCC)
- net CLOCK: now also U5.11 (SRCLK)
- net GND: now also U5.8 (GND)
- net LATCH: now also U5.12 (RCLK)
- net OE: now also U5.13 (~{OE})
- net RESET: now also U5.10 (~{SRCLR})
- net SIN: now also U5.14 (SER)
- net SOUT: now also U5.9 (QH')
- net at R89.2, R90.2: now also U5.4 (QE)
- net at R91.2, R92.2: now also U5.5 (QF)
- net at R93.2, R94.2: now also U5.6 (QG)
- net at R95.2, R96.2: now also U5.7 (QH)
- net at R87.2, R88.2: now also U5.3 (QD)
- net at R85.2, R86.2: now also U5.2 (QC)
- net at R83.2, R84.2: now also U5.1 (QB)
- net at R81.2, R82.2: now also U5.15 (QA)
