File: Hardware/Electronics/Schematic/MainBoard/MainBoard.kicad_sch (KiCad schematic)
At the start: 67 parts, among them P10 AUX, P2 CONN_02X08, P3 SWD/JTAG, P4 BUTTON1, P6 BUTTON3, P7 BUTTON4, P8 POWER_IN, P9 DEBUG_UART, SW1 STM_RESET, SW2 ESP_RESET, SW3 ESP_PROG, U10 S25FL129P, U11 MAX9700, U15 TPS6211, U9 ESP-12F, Y1 8MHz, Y2 32.768kHz

Commit message: Kicad files cleanup
Parts:
- gave numbers to parts that had none: 6
